File: Datalogger.brd (EAGLE design)
At the start: 90 x 53.8 mm, 30 parts, among them IC1 7805T, IC2 MEGA8-AI, U1 DS1307Z, X1 32.768KHZ

Commit message: ground plane completed
Parts:
- moved L1 133.9 mm to (61.7, 22.4)
- moved C7 108.8 mm to (61.6, 27.3)
- moved CN1 105.8 mm to (80.3, -2.29)
- moved Q1 99.9 mm to (38.0, 23.4), turned to 270 degrees
- moved X4 93.7 mm to (45.0, 5.08)
- moved C9 93.3 mm to (39.4, 32.8)
- moved X3 93.1 mm to (61.1, 5.71)
- moved C6 85.2 mm to (33.0, 20.8)
- moved IC2 83.4 mm to (50.2, 28.2)
- moved X5 81.1 mm to (13.5, 4.83)
- moved X2 80.2 mm to (29.3, 4.83)
- moved C5 78.9 mm to (33.0, 26.2)
- moved C10 73.7 mm to (44.6, 34.9)
- moved C1 1.80 mm to (81.0, 19.8)
- moved C3 1.66 mm to (86.2, 27.4)
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Connections:
- removed net N$6: C10.1, C9.1, IC2.4, IC2.6
- net VCC: now also C10.1, C9.1, IC2.4, IC2.6
Routing:
- net GND: track 0.00 -> 31.4 mm
- net N$1: track 0.00 -> 19.4 mm
- added copper zone on layer 1, net GND

Commit message: component value updated
Parts:
- C1, C2: value (none) -> 100u
- C10, C4, C7, C8: value (none) -> 0.1u
- C3: value (none) -> 0.1
- C5, C6: value (none) -> 22p
- C9: value (none) -> 0.01u
- L1: value (none) -> 100m
- Q1: value (none) -> 16M
- R1: value (none) -> 10k
Changed lines of the file:
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@@
 <attribute name="VALUE" x="-29.21" y="26.67" size="1.27" layer="27" ratio="10"/>
 </element>
-<element name="C1" library="rcl" library_urn="urn:adsk.eagle:library:334" package="140CLH-1010" package3d_urn="urn:adsk.eagle:package:23391/2" value="" x="80.95" y="19.77" smashed="yes">
+<element name="C1" library="rcl" library_urn="urn:adsk.eagle:library:334" package="140CLH-1010" package3d_urn="urn:adsk.eagle:package:23391/2" value="100u" x="80.95" y="19.77" smashed="yes">
 <attribute name="NAME" x="78.21" y="21.7" size="1.27" layer="25"/>
 <attribute name="POPULARITY" value="0" x="101.27" y="-43.73" size="1.778" layer="27" display="off"/>
@@
 <attribute name="VALUE" x="77.575" y="16.885" size="1.27" layer="27"/>
 </element>
-<element name="C10" library="rcl" library_urn="urn:adsk.eagle:library:334" package="C0603" package3d_urn="urn:adsk.eagle:package:23616/2" value="" x="44.577" y="34.925" smashed="yes">
+<element name="C10" library="rcl" library_urn="urn:adsk.eagle:library:334" package="C0603" package3d_urn="urn:adsk.eagle:package:23616/2" value="0.1u" x="44.577" y="34.925" smashed="yes">
 <attribute name="NAME" x="43.942" y="35.56" size="1.27" layer="25"/>
 <attribute name="POPULARITY" value="73" x="61.087" y="-41.275" size="1.778" layer="27" display="off"/>
@@
 <attribute name="VALUE" x="-60.325" y="70.485" size="1.27" layer="27"/>
 </element>
-<element name="C2" library="rcl" library_urn="urn:adsk.eagle:library:334" package="140CLH-1010" package3d_urn="urn:adsk.eagle:package:23391/2" value="" x="-34.29" y="63.5" smashed="yes">
+<element name="C2" library="rcl" library_urn="urn:adsk.eagle:library:334" package="140CLH-1010" package3d_urn="urn:adsk.eagle:package:23391/2" value="100u" x="-34.29" y="63.5" smashed="yes">
 <attribute name="NAME" x="-37.03" y="65.43" size="1.27" layer="25"/>
 <attribute name="POPULARITY" value="0" x="0" y="0" size="1.778" layer="27" display="off"/>
@@
 <attribute name="VALUE" x="-37.665" y="60.615" size="1.27" layer="27"/>
 </element>
-<element name="C3" library="rcl" library_urn="urn:adsk.eagle:library:334" package="C0603" package3d_urn="urn:adsk.eagle:package:23616/2" value="" x="86.209" y="27.403" smashed="yes" rot="R180">
+<element name="C3" library="rcl" library_urn="urn:adsk.eagle:library:334" package="C0603" package3d_urn="urn:adsk.eagle:package:23616/2" value="0.1" x="86.209" y="27.403" smashed="yes" rot="R180">
 <attribute name="NAME" x="86.844" y="26.768" size="1.27" layer="25" rot="R180"/>
 <attribute name="POPULARITY" value="73" x="65.889" y="103.603" size="1.778" layer="27" rot="R180" display="off"/>
@@
 <attribute name="VALUE" x="86.844" y="29.308" size="1.27" layer="27" rot="R180"/>
 </element>
-<element name="C4" library="rcl" library_urn="urn:adsk.eagle:library:334" package="C0603" package3d_urn="urn:adsk.eagle:package:23616/2" value="" x="-24.13" y="76.2" smashed="yes">
+<element name="C4" library="rcl" library_urn="urn:adsk.eagle:library:334" package="C0603" package3d_urn="urn:adsk.eagle:package:23616/2" value="0.1u" x="-24.13" y="76.2" smashed="yes">
 <attribute name="NAME" x="-24.765" y="76.835" size="1.27" layer="25"/>
 <attribute name="POPULARITY" value="73" x="0" y="0" size="1.778" layer="27" display="off"/>
@@
 <attribute name="VALUE" x="-24.765" y="74.295" size="1.27" layer="27"/>
 </element>
-<element name="C5" library="rcl" library_urn="urn:adsk.eagle:library:334" package="C0603" package3d_urn="urn:adsk.eagle:package:23616/2" value="" x="33.02" y="26.162" smashed="yes">
+<element name="C5" library="rcl" library_urn="urn:adsk.eagle:library:334" package="C0603" package3d_urn="urn:adsk.eagle:package:23616/2" value="22p" x="33.02" y="26.162" smashed="yes">
 <attribute name="NAME" x="32.385" y="26.797" size="1.27" layer="25"/>
 <attribute name="POPULARITY" value="73" x="60.96" y="-50.038" size="1.778" layer="27" display="off"/>
@@
 <attribute name="VALUE" x="32.385" y="24.257" size="1.27" layer="27"/>
 </element>
-<element name="C6" library="rcl" library_urn="urn:adsk.eagle:library:334" package="C0603" package3d_urn="urn:adsk.eagle:package:23616/2" value="" x="33.02" y="20.828" smashed="yes">
+<element name="C6" library="rcl" library_urn="urn:adsk.eagle:library:334" package="C0603" package3d_urn="urn:adsk.eagle:package:23616/2" value="22p" x="33.02" y="20.828" smashed="yes">
 <attribute name="NAME" x="32.385" y="21.463" size="1.27" layer="25"/>
 <attribute name="POPULARITY" value="73" x="64.77" y="-55.372" size="1.778" layer="27" display="off"/>
@@
 <attribute name="VALUE" x="32.385" y="18.923" size="1.27" layer="27"/>
 </element>
-<element name="C7" library="rcl" library_urn="urn:adsk.eagle:library:334" package="C0603" package3d_urn="urn:adsk.eagle:package:23616/2" value="" x="61.595" y="27.305" smashed="yes">
+<element name="C7" library="rcl" library_urn="urn:adsk.eagle:library:334" package="C0603" package3d_urn="urn:adsk.eagle:package:23616/2" value="0.1u" x="61.595" y="27.305" smashed="yes">
 <attribute name="NAME" x="60.96" y="27.94" size="1.27" layer="25"/>
 <attribute name="POPULARITY" value="73" x="97.155" y="-48.895" size="1.778" layer="27" display="off"/>
@@
 <attribute name="VALUE" x="60.96" y="25.4" size="1.27" layer="27"/>
 </element>
-<element name="C8" library="rcl" library_urn="urn:adsk.eagle:library:334" package="C0603" package3d_urn="urn:adsk.eagle:package:23616/2" value="" x="-39.37" y="76.2" smashed="yes">
+<element name="C8" library="rcl" library_urn="urn:adsk.eagle:library:334" package="C0603" package3d_urn="urn:adsk.eagle:package:23616/2" value="0.1u" x="-39.37" y="76.2" smashed="yes">
 <attribute name="NAME" x="-40.005" y="76.835" size="1.27" layer="25"/>
 <attribute name="POPULARITY" value="73" x="0" y="0" size="1.778" layer="27" display="off"/>
@@
 <attribute name="VALUE" x="-40.005" y="74.295" size="1.27" layer="27"/>
 </element>
-<element name="C9" library="rcl" library_urn="urn:adsk.eagle:library:334" package="C0603" package3d_urn="urn:adsk.eagle:package:23616/2" value="" x="39.37" y="32.766" smashed="yes">
+<element name="C9" library="rcl" library_urn="urn:adsk.eagle:library:334" package="C0603" package3d_urn="urn:adsk.eagle:package:23616/2" value="0.01u" x="39.37" y="32.766" smashed="yes">
 <attribute name="NAME" x="38.735" y="33.401" size="1.27" layer="25"/>
 <attribute name="POPULARITY" value="73" x="82.55" y="-43.434" size="1.778" layer="27" display="off"/>
@@
 <attribute name="VALUE" x="47.1424" y="26.924" size="0.8128" layer="27"/>
 </element>
-<element name="L1" library="rcl" library_urn="urn:adsk.eagle:library:334" package="L2012C" package3d_urn="urn:adsk.eagle:package:23475/2" value="" x="61.722" y="22.352" smashed="yes">
+<element name="L1" library="rcl" library_urn="urn:adsk.eagle:library:334" package="L2012C" package3d_urn="urn:adsk.eagle:package:23475/2" value="100m" x="61.722" y="22.352" smashed="yes">
 <attribute name="NAME" x="59.817" y="23.622" size="1.27" layer="25"/>
 <attribute name="POPULARITY" value="6" x="125.222" y="-47.498" size="1.778" layer="27" display="off"/>
@@
 <attribute name="VALUE" x="59.817" y="19.812" size="1.27" layer="27"/>
 </element>
-<element name="Q1" library="special" library_urn="urn:adsk.eagle:library:367" package="QS" package3d_urn="urn:adsk.eagle:package:26647/2" value="" x="37.973" y="23.368" smashed="yes" rot="R270">
+<element name="Q1" library="special" library_urn="urn:adsk.eagle:library:367" package="QS" package3d_urn="urn:adsk.eagle:package:26647/2" value="16M" x="37.973" y="23.368" smashed="yes" rot="R270">
 <attribute name="NAME" x="40.64" y="28.448" size="1.27" layer="25" ratio="10" rot="R270"/>
 <attribute name="POPULARITY" value="59" x="-22.987" y="-31.242" size="1.778" layer="27" rot="R270" display="off"/>
 <attribute name="VALUE" x="34.036" y="28.448" size="1.27" layer="27" ratio="10" rot="R270"/>
 </element>
-<element name="R1" library="rcl" library_urn="urn:adsk.eagle:library:334" package="R0603" package3d_urn="urn:adsk.eagle:package:23555/3" value="" x="-46.99" y="76.2" smashed="yes">
+<element name="R1" library="rcl" library_urn="urn:adsk.eagle:library:334" package="R0603" package3d_urn="urn:adsk.eagle:package:23555/3" value="10k" x="-46.99" y="76.2" smashed="yes">
 <attribute name="NAME" x="-47.625" y="76.835" size="1.27" layer="25"/>
 <attribute name="POPULARITY" value="77" x="0" y="0" size="1.778" layer="27" display="off"/>
